File: hardware/main_board/controls_lcd.kicad_sch (KiCad schematic)
At the start: 28 parts, among them J6 2434804-1, Q1 AO3400A, Q2 AO3400A, Q3 AO3400A, Q4 AO3401A, SW3 SW_Push, U5 NHD-C0220BIZ-FSRGB

Commit message: Route 4-layer PCB
Connections:
- net GND: now also SW3.2; no longer SW3.1
- net at R17.1: now also SW3.1; no longer SW3.2
Changed lines of the file:
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@@
 		(lib_id "Switch:SW_Push")
 		(at 58.42 107.95 0)
+		(mirror y)
 		(unit 1)
 		(exclude_from_sim no)
@@
 		(on_board yes)
 		(dnp no)
-		(fields_autoplaced yes)
 		(property "Reference" "SW3"
 			(at 58.42 100.33 0)
