File: hardware/main_board/main_board.kicad_pcb (KiCad board)
At the start: 2 copper layers, 77 x 57.2 mm, 69 parts, among them J1 USB_C_Receptacle_USB2.0_16P, J2 Conn_01x03, J3 Conn_01x03, J4 Conn_02x05_Odd_Even, J5 Conn_02x10_Odd_Even, J6 2434804-1, Q1 AO3400A, Q2 AO3400A, Q3 AO3400A, Q4 AO3401A, SW1 SW_Push, SW2 SW_Push, SW3 SW_Push, U1 USBLC6-2SC6, U2 BQ24259RGER, U3 TPS7A0533PDBV, U4 STM32G0B1CBTx, U5 NHD-C0220BIZ-FSRGB

Commit message: Route 4-layer PCB
Parts:
- moved C11 44.4 mm to (99.2, 59.0), turned to 180 degrees
- moved C18 36.7 mm to (108.2, 54.1), turned to 90 degrees
- moved C17 34.4 mm to (112.0, 57.4)
- moved C16 32.7 mm to (109.4, 54.1), turned to 90 degrees
- moved C20 31.5 mm to (112.0, 55.0), turned to 180 degrees
- moved C15 30.7 mm to (112.0, 58.6)
- moved C19 28.0 mm to (112.0, 56.2), turned to 0 degrees
- moved R16 9.29 mm to (115.2, 84.3), turned to 90 degrees
- moved R14 6.47 mm to (113.8, 84.3), turned to -90 degrees
- moved R15 3.73 mm to (112.4, 84.3), turned to -90 degrees
- moved R17 3.20 mm to (101.6, 88.8), turned to 0 degrees
- moved R18 2.25 mm to (121.0, 84.3), turned to -90 degrees
- moved D1 2.25 mm to (66.2, 85.0)
- moved R4 2.25 mm to (69.2, 85.0)
- moved D2 2.20 mm to (66.2, 87.2)
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Connections:
- J4 pad 1: /MCU/3V3 -> /MCU/NRST
- J4 pad 10: /MCU/NRST -> /MCU/3V3
- J4 pad 2: /MCU/SYS_SWDIO -> unconnected-(J4-Pin_2-Pad2)
- J4 pad 3: GND -> unconnected-(J4-Pin_3-Pad3)
- J4 pad 4: /MCU/SYS_SWCLK -> unconnected-(J4-Pin_4-Pad4)
- J4 pad 5: GND -> unconnected-(J4-Pin_5-Pad5)
- J4 pad 6: unconnected-(J4-Pin_6-Pad6) -> GND
- J4 pad 7: unconnected-(J4-Pin_7-Pad7) -> /MCU/SYS_SWCLK
- J4 pad 8: unconnected-(J4-Pin_8-Pad8) -> GND
- J4 pad 9: unconnected-(J4-Pin_9-Pad9) -> /MCU/SYS_SWDIO
- SW3 pad 1: GND -> Net-(R17-Pad1)
- SW3 pad 2: Net-(R17-Pad1) -> GND
- U1 pad 1: /MCU/D- -> /MCU/D+
- U1 pad 3: /MCU/D+ -> /MCU/D-
- U1 pad 4: /Power/USBCONN_D+ -> /Power/USBCONN_D-
- U1 pad 6: /Power/USBCONN_D- -> /Power/USBCONN_D+
- U4 pad 22: /MCU/DIR_D -> /MCU/BUTTON
- U4 pad 23: /MCU/DIR_B -> /MCU/DIR_A
- U4 pad 24: /MCU/DIR_A -> /MCU/DIR_D
- U4 pad 25: /MCU/CENTER -> /MCU/DIR_B
- U4 pad 27: /MCU/BUTTON -> /MCU/CENTER
Routing:
- net /MCU/3V3: track 199.1 -> 4.61 mm, vias 2 -> 7
- net GND: track 57.1 -> 68.7 mm, vias 28 -> 26
- net /MCU/CENTER: track 38.7 -> 28.1 mm
- net /MCU/DIR_C: track 40.0 -> 30.2 mm
- net /MCU/NRST: track 66.5 -> 56.9 mm, vias 4 -> 2
- net Net-(U2-REGN): track 26.1 -> 16.5 mm
- net /MCU/DIR_D: track 43.0 -> 37.2 mm
- net /MCU/D+: track 61.2 -> 55.8 mm, vias 6 -> 2
- net /MCU/D-: track 61.1 -> 55.9 mm, vias 6 -> 2
- net /MCU/DIR_A: track 38.3 -> 33.4 mm
- net Net-(J6-C): track 3.75 -> 8.41 mm
- net Net-(J6-CENTER): track 3.26 -> 7.57 mm
- net /MCU/VBUS: track 117.5 -> 113.4 mm, vias 0 -> 5
- net /MCU/SDA: track 84.5 -> 80.5 mm, vias 4 -> 1
- net /MCU/DIR_B: track 38.1 -> 34.1 mm
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- added copper zone on In1.Cu, net /MCU/3V3
- added copper zone on In2.Cu, net GND
- removed copper zone on F.Cu, net GND
Other:
- copper layers 2 -> 4

Commit message: Add SYS power to the extension socket
Connections:
- J5 pad 19: GND -> /Power/SYS
Routing:
- net /Power/SYS: track 54.1 -> 156.6 mm, vias 3 -> 4
- net GND: vias 26 -> 25
Changed lines of the file:
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@@
 			(size 1.02 2.285)
 			(layers "B.Cu" "B.Mask" "B.Paste")
-			(net 1 "GND")
+			(net 8 "/Power/SYS")
 			(pinfunction "Pin_19")
 			(pintype "passive")
@@
 	)
 	(via
-		(at 126.105 68.2)
-		(size 0.8)
-		(drill 0.4)
-		(layers "F.Cu" "B.Cu")
-		(net 1)
-	)
-	(via
 		(at 79.21 56.025)
 		(size 0.8)
@@
 	)
 	(segment
-		(start 87.148378 99)
-		(end 136.4 99)
+		(start 136.4 99)
+		(end 137.85 97.55)
 		(width 0.5)
 		(layer "In1.Cu")
@@
 	)
 	(segment
-		(start 137.4 70.1)
+		(start 137.85 70.55)
 		(end 135.5 68.2)
 		(width 0.5)
@@
 	)
 	(segment
-		(start 137.4 98)
-		(end 137.4 70.1)
-		(width 0.5)
-		(layer "In1.Cu")
-		(net 3)
-	)
-	(segment
 		(start 73.2875 93.4125)
 		(end 75.300811 95.425811)
@@
 	)
 	(segment
-		(start 136.4 99)
-		(end 137.4 98)
+		(start 83.574189 95.425811)
+		(end 87.148378 99)
 		(width 0.5)
 		(layer "In1.Cu")
@@
 	)
 	(segment
-		(start 83.574189 95.425811)
-		(end 87.148378 99)
+		(start 137.85 97.55)
+		(end 137.85 70.55)
+		(width 0.5)
+		(layer "In1.Cu")
+		(net 3)
+	)
+	(segment
+		(start 87.148378 99)
+		(end 136.4 99)
 		(width 0.5)
 		(layer "In1.Cu")
@@
 	)
 	(via
+		(at 126.105 68.2)
+		(size 0.8)
+		(drill 0.4)
+		(layers "F.Cu" "B.Cu")
+		(net 8)
+	)
+	(via
 		(at 65.3125 85)
 		(size 0.8)
@@
 	)
 	(segment
+		(start 135.95 98.05)
+		(end 92.2 98.05)
+		(width 0.5)
+		(layer "In1.Cu")
+		(net 8)
+	)
+	(segment
+		(start 136.85 78.95)
+		(end 136.85 97.15)
+		(width 0.5)
+		(layer "In1.Cu")
+		(net 8)
+	)
+	(segment
 		(start 82.560315 84)
 		(end 83.612448 82.947867)
@@
 	)
 	(segment
+		(start 136.85 97.15)
+		(end 135.95 98.05)
+		(width 0.5)
+		(layer "In1.Cu")
+		(net 8)
+	)
+	(segment
+		(start 91.2 97.05)
+		(end 91.2 82.45)
+		(width 0.5)
+		(layer "In1.Cu")
+		(net 8)
+	)
+	(segment
 		(start 66.3125 84)
 		(end 82.560315 84)
@@
 	(segment
 		(start 83.612448 82.947867)
-		(end 83.612448 65.862448)
+		(end 83.612448 81.2)
 		(width 0.5)
 		(layer "In1.Cu")
@@
 	)
 	(segment
+		(start 91.2 82.45)
+		(end 89.95 81.2)
+		(width 0.5)
+		(layer "In1.Cu")
+		(net 8)
+	)
+	(segment
+		(start 89.95 81.2)
+		(end 83.612448 81.2)
+		(width 0.5)
+		(layer "In1.Cu")
+		(net 8)
+	)
+	(segment
+		(start 126.105 68.2)
+		(end 126.105 68.205)
+		(width 0.5)
+		(layer "In1.Cu")
+		(net 8)
+	)
+	(segment
+		(start 126.105 68.205)
+		(end 136.85 78.95)
+		(width 0.5)
+		(layer "In1.Cu")
+		(net 8)
+	)
+	(segment
+		(start 83.612448 81.2)
+		(end 83.612448 65.862448)
+		(width 0.5)
+		(layer "In1.Cu")
+		(net 8)
+	)
+	(segment
+		(start 92.2 98.05)
+		(end 91.2 97.05)
+		(width 0.5)
+		(layer "In1.Cu")
+		(net 8)
+	)
+	(segment
 		(start 83.612448 65.862448)
 		(end 83 65.25)
@@
 		(polygon
 			(pts
-				(xy 136.2 98.1) (xy 136.2 43.6) (xy 62.2 43.6) (xy 62.2 69.2) (xy 79 69.2) (xy 79 63.7) (xy 92.5 63.7)
-				(xy 92.5 98.1)
+				(xy 134.85 97.35) (xy 134.85 43.6) (xy 62.2 43.6) (xy 62.2 69.2) (xy 79 69.2) (xy 79 63.7) (xy 92.5 63.7)
+				(xy 92.5 97.35)
 			)
 		)

Commit message: Add expansion socket markings
Other:
- board text added: "3V3"
- board text added: "GND"
- board text added: "SCL"
- board text added: "SDA"
- board text added: "SYS"
- board text added: "VBUS"
Changed lines of the file:
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@@
+		)
+	)
+	(gr_text "SCL"
+		(at 119.65 66.26175 0)
+		(layer "B.SilkS")
+		(effects
+			(font
+				(size 1 1)
+				(thickness 0.15)
+			)
+			(justify left bottom mirror)
+		)
+	)
+	(gr_text "SDA"
+		(at 124.3 66.26175 0)
+		(layer "B.SilkS")
+		(effects
+			(font
+				(size 1 1)
+				(thickness 0.15)
+			)
+			(justify left bottom mirror)
+		)
+	)
+	(gr_text "3V3"
+		(at 119.65 45.94175 0)
+		(layer "B.SilkS")
+		(effects
+			(font
+				(size 1 1)
+				(thickness 0.15)
+			)
+			(justify left bottom mirror)
+		)
+	)
+	(gr_text "SYS"
+		(at 119.65 68.80175 0)
+		(layer "B.SilkS")
+		(effects
+			(font
+				(size 1 1)
+				(thickness 0.15)
+			)
+			(justify left bottom mirror)
+		)
+	)
+	(gr_text "GND"
+		(at 124.3 45.94175 0)
+		(layer "B.SilkS")
+		(effects
+			(font
+				(size 1 1)
+				(thickness 0.15)
+			)
+			(justify left bottom mirror)
+		)
+	)
+	(gr_text "VBUS"
+		(at 124.3 68.80175 0)
+		(layer "B.SilkS")
+		(effects
+			(font
+				(size 1 1)
+				(thickness 0.15)
+			)
+			(justify left bottom mirror)
 		)
 	)
